Commit message: fixing urdf

File: src/projeto/urdf/macros/parts/camera.urdf.xacro (robot description, xacro)
@@ -2,5 +2,5 @@
 <robot xmlns:xacro="http://ros.org/wiki/xacro">
   <xacro:macro name="camera" params="name parent x y z">
-    <!-- joint: base_footprint -> base -->
+    <!-- joint: camera -> screen -->
     <joint name="${parent}_to_${name}" type="fixed">
       <origin xyz="${x} ${y} ${z}" rpy="0 0 0"/>

File: src/projeto/urdf/macros/parts/holder.urdf.xacro (robot description, xacro)
@@ -1,5 +1,5 @@
 <?xml version="1.0"?>
 <robot xmlns:xacro="http://ros.org/wiki/xacro">
-  <xacro:macro name="holder" params="name parent1 parent2 x y z">
+  <xacro:macro name="holder" params="name parent child x y z">
     <!-- joint: plate -> holder -->
       <joint name="${parent1}_to_${name}" type="fixed">
@@ -9,7 +9,7 @@
       </joint>
       <joint name="${name}_to_${parent2}" type="fixed">
-        <origin xyz="${x} ${y} -${z}" rpy="0 0 0"/>
-        <parent link="${parent2}"/>
-        <child link="${name}"/>
+        <origin xyz="${-1*x} ${-1*y} ${z}" rpy="0 0 0"/>
+        <parent link="${name}"/>
+        <child link="${child}"/>
       </joint>
     <!-- link: base -->

File: src/projeto/urdf/macros/parts/screen.urdf.xacro (robot description, xacro)
@@ -2,5 +2,5 @@
 <robot xmlns:xacro="http://ros.org/wiki/xacro">
   <xacro:macro name="screen" params="name x y z">
-    <!-- joint: base_footprint -> base -->
+    <!-- joint: screen -> plate -->
     <joint name="plate_top_to_${name}" type="fixed">
       <origin xyz="${x} ${y} ${z}" rpy="0 0 0"/>

File: src/projeto/urdf/macros/parts/torso.urdf.xacro (robot description, xacro)
@@ -2,5 +2,5 @@
 <robot xmlns:xacro="http://ros.org/wiki/xacro">
   <xacro:macro name="torso" params="name">
-    <!-- joint: base_footprint -> base -->
+    <!-- joint: torso -> laser -->
     <joint name="torso_to_laser" type="fixed">
       <origin xyz="0 0 0.2125" rpy="0 0 0"/>
@@ -14,5 +14,5 @@
       </xacro:create_cylinder>
     </link>
-    <!-- joint: base_footprint -> base -->
+    <!-- joint: torso -> laser -->
       <joint name="torso_to_plate" type="fixed">
         <origin xyz="0 0 0.21" rpy="0 0 0"/>

File: src/projeto/urdf/robot.urdf.xacro (robot description, xacro)
@@ -20,12 +20,12 @@
   <xacro:plate name="plate_middle"/>
   <xacro:plate name="plate_top"/>
-  <xacro:holder name="holder1" parent1="plate_bottom" parent2="plate_middle" x= "${holder_xy}" y="${holder_xy}" z="${holder_z}"/>
-  <xacro:holder name="holder2" parent1="plate_bottom" parent2="plate_middle" x= "-${holder_xy}" y="-${holder_xy}" z="${holder_z}"/>
-  <xacro:holder name="holder3" parent1="plate_bottom" parent2="plate_middle" x= "-${holder_xy}" y="${holder_xy}" z="${holder_z}"/>
-  <xacro:holder name="holder4" parent1="plate_bottom" parent2="plate_middle" x= "${holder_xy}" y="-${holder_xy}" z="${holder_z}"/>
-  <xacro:holder name="holder5" parent1="plate_middle" parent2="plate_top" x= "${holder_xy}" y="${holder_xy}" z="${holder_z}"/>
-  <xacro:holder name="holder6" parent1="plate_middle" parent2="plate_top" x= "-${holder_xy}" y="-${holder_xy}" z="${holder_z}"/>
-  <xacro:holder name="holder7" parent1="plate_middle" parent2="plate_top" x= "-${holder_xy}" y="${holder_xy}" z="${holder_z}"/>
-  <xacro:holder name="holder8" parent1="plate_middle" parent2="plate_top" x= "${holder_xy}" y="-${holder_xy}" z="${holder_z}"/>
+  <xacro:holder name="holder1" parent="plate_bottom" child="plate_middle" x= "${holder_xy}" y="${holder_xy}" z="${holder_z}"/>
+  <xacro:holder name="holder2" parent="plate_bottom" child="plate_middle" x= "${-1*holder_xy}" y="-${-1*holder_xy}" z="${holder_z}"/>
+  <xacro:holder name="holder3" parent="plate_bottom" child="plate_middle" x= "${-1*holder_xy}" y="${holder_xy}" z="${holder_z}"/>
+  <xacro:holder name="holder4" parent="plate_bottom" child="plate_middle" x= "${holder_xy}" y="${-1*holder_xy}" z="${holder_z}"/>
+  <xacro:holder name="holder5" parent="plate_middle" child="plate_top" x= "${holder_xy}" y="${holder_xy}" z="${holder_z}"/>
+  <xacro:holder name="holder6" parent="plate_middle" child="plate_top" x= "${-1*holder_xy}" y="${-1*holder_xy}" z="${holder_z}"/>
+  <xacro:holder name="holder7" parent="plate_middle" child="plate_top" x= "${-1*holder_xy}" y="${holder_xy}" z="${holder_z}"/>
+  <xacro:holder name="holder8" parent="plate_middle" child="plate_top" x= "${holder_xy}" y="${-1*holder_xy}" z="${holder_z}"/>
   <xacro:screen name="screen_front" x="0.18" y="0" z="0.02"/>
   <xacro:screen name="screen_back" x="-0.18" y="0" z="0.02"/>
