Commit message: fixing urdf

File: src/projeto/urdf/macros/parts/holder.urdf.xacro (robot description, xacro)
@@ -9,7 +9,7 @@
       </joint>
       <joint name="${name}_to_${parent2}" type="fixed">
-        <origin xyz="-${x} -${y} ${z}" rpy="0 0 0"/>
-        <parent link="${name}"/>
-        <child link="${parent2}"/>
+        <origin xyz="${x} ${y} -${z}" rpy="0 0 0"/>
+        <parent link="${parent2}"/>
+        <child link="${name}"/>
       </joint>
     <!-- link: base -->

Commit message: fixing urdf

File: src/projeto/urdf/macros/parts/holder.urdf.xacro (robot description, xacro)
@@ -5,5 +5,5 @@
       <joint name="${parent1}_to_${name}" type="fixed">
         <origin xyz="${x} ${y} ${z}" rpy="0 0 0"/>
-        <parent link="${parent1}"/>
+        <parent link="${parent}"/>
         <child link="${name}"/>
       </joint>

Commit message: fixing urdf

File: src/projeto/urdf/macros/parts/holder.urdf.xacro (robot description, xacro)
@@ -3,10 +3,10 @@
   <xacro:macro name="holder" params="name parent child x y z">
     <!-- joint: plate -> holder -->
-      <joint name="${parent1}_to_${name}" type="fixed">
+      <joint name="${parent}_to_${name}" type="fixed">
         <origin xyz="${x} ${y} ${z}" rpy="0 0 0"/>
         <parent link="${parent}"/>
         <child link="${name}"/>
       </joint>
-      <joint name="${name}_to_${parent2}" type="fixed">
+      <joint name="${name}_to_${child}" type="fixed">
         <origin xyz="${-1*x} ${-1*y} ${z}" rpy="0 0 0"/>
         <parent link="${name}"/>

Commit message: finalizando mapping

File: src/projeto/urdf/macros/parts/holder.urdf.xacro (robot description, xacro)
@@ -1,13 +1,13 @@
 <?xml version="1.0"?>
 <robot xmlns:xacro="http://ros.org/wiki/xacro">
-  <xacro:macro name="holder" params="name parent child x y z">
+  <xacro:macro name="holder" params="name parent child z">
     <!-- joint: plate -> holder -->
       <joint name="${parent}_to_${name}" type="fixed">
-        <origin xyz="${x} ${y} ${z}" rpy="0 0 0"/>
+        <origin xyz="0 0 ${z}" rpy="0 0 0"/>
         <parent link="${parent}"/>
         <child link="${name}"/>
       </joint>
       <joint name="${name}_to_${child}" type="fixed">
-        <origin xyz="${-1*x} ${-1*y} ${z}" rpy="0 0 0"/>
+        <origin xyz="0 0 ${z}" rpy="0 0 0"/>
         <parent link="${name}"/>
         <child link="${child}"/>
@@ -16,5 +16,14 @@
     <link name="${name}">
       <xacro:create_cylinder m="${holder_mass}" r="${holder_radius}" l="${holder_length}">
-        <origin xyz="0 0 0" rpy="0 0 0"/>
+        <origin xyz="${holder_xy} ${holder_xy} 0" rpy="0 0 0"/>
+      </xacro:create_cylinder>
+      <xacro:create_cylinder m="${holder_mass}" r="${holder_radius}" l="${holder_length}">
+        <origin xyz="${-1*holder_xy} ${-1*holder_xy} 0" rpy="0 0 0"/>
+      </xacro:create_cylinder>
+      <xacro:create_cylinder m="${holder_mass}" r="${holder_radius}" l="${holder_length}">
+        <origin xyz="${holder_xy} ${-1*holder_xy} 0" rpy="0 0 0"/>
+      </xacro:create_cylinder>
+      <xacro:create_cylinder m="${holder_mass}" r="${holder_radius}" l="${holder_length}">
+        <origin xyz="${-1*holder_xy} ${holder_xy} 0" rpy="0 0 0"/>
       </xacro:create_cylinder>
     </link>

File: src/projeto/urdf/macros/parts/screen.urdf.xacro (robot description, xacro)
@@ -1,9 +1,9 @@
 <?xml version="1.0"?>
 <robot xmlns:xacro="http://ros.org/wiki/xacro">
-  <xacro:macro name="screen" params="name x y z">
+  <xacro:macro name="screen" params="name parent x y z">
     <!-- joint: screen -> plate -->
     <joint name="plate_top_to_${name}" type="fixed">
       <origin xyz="${x} ${y} ${z}" rpy="0 0 0"/>
-      <parent link="plate_top"/>
+      <parent link="${parent}"/>
       <child link="${name}"/>
     </joint>

File: src/projeto/urdf/macros/parts/torso.urdf.xacro (robot description, xacro)
@@ -1,9 +1,9 @@
 <?xml version="1.0"?>
 <robot xmlns:xacro="http://ros.org/wiki/xacro">
-  <xacro:macro name="torso" params="name">
+  <xacro:macro name="torso" params="name parent child">
     <!-- joint: torso -> laser -->
     <joint name="torso_to_laser" type="fixed">
       <origin xyz="0 0 0.2125" rpy="0 0 0"/>
-      <parent link="base_scan"/>
+      <parent link="${parent}"/>
       <child link="${name}"/>
     </joint>
@@ -18,5 +18,5 @@
         <origin xyz="0 0 0.21" rpy="0 0 0"/>
         <parent link="${name}"/>
-        <child link="plate_bottom"/>
+        <child link="${child}"/>
       </joint>
   </xacro:macro>

File: src/projeto/urdf/macros/properties.urdf.xacro (robot description, xacro)
@@ -23,5 +23,5 @@
   <xacro:property name="camera_mass"      value="${2 * robot_mass/100}" />
   <xacro:property name="camera_x"         value="0.025" />
-  <xacro:property name="camera_y"         value="0.2" />
+  <xacro:property name="camera_y"         value="0.025" />
   <xacro:property name="camera_z"         value="0.02" />
   <xacro:property name="wheel_mass"      value="${5 * robot_mass/100}" />

File: src/projeto/urdf/robot.urdf (robot description, URDF)
Before this commit: robot garcom, 20 links, 25 joints
Links:
- removed link base
- removed link holder_1
- removed link holder_2
- removed link holder_3
- removed link holder_4
- removed link holder_5
- removed link holder_6
- removed link holder_7
- removed link holder_8
- added link base_link, mass 2.0; collision cylinder length=0.4 radius=0.2; visual cylinder length=0.4 radius=0.2
- added link camera_frente, mass 0.2; collision box size=0.025 0.025 0.02; visual box size=0.025 0.025 0.02
- added link holder1, mass 0.125; collision cylinder length=0.2 radius=0.02; collision cylinder length=0.2 radius=0.02
- added link holder2, mass 0.125; collision cylinder length=0.2 radius=0.02; collision cylinder length=0.2 radius=0.02
- added link imu, mass 1e-5; collision box size=0.2 0.2 0.05; visual box size=0.2 0.2 0.05
- link base_scan: mass 1 -> 1.0; geometry collision cylinder length=0.025 radius=0.2; visual cylinder length=0.025 radius=0.2
- link front_wheel: mass 0.25 -> 0.5; geometry collision sphere radius=0.06666666666666667; visual sphere radius=0.06666666666666667
- link left_wheel: mass 0.25 -> 0.5; geometry collision sphere radius=0.06666666666666667; visual sphere radius=0.06666666666666667
- link plate_bottom: mass 1 -> 0.5
- link plate_middle: mass 1 -> 0.5
- link plate_top: mass 1 -> 0.5
- link right_wheel: mass 0.25 -> 0.5; geometry collision sphere radius=0.06666666666666667; visual sphere radius=0.06666666666666667
- link screen_back: mass 1 -> 0.4
- link screen_front: mass 1 -> 0.4
- link torso: mass 1 -> 2.0; geometry collision cylinder length=0.4 radius=0.2; visual cylinder length=0.4 radius=0.2
Joints:
- removed joint joint_base_scan_to_torso
- removed joint joint_base_to_base_scan
- removed joint joint_base_to_front_wheel
- removed joint joint_base_to_left_wheel
- removed joint joint_base_to_right_wheel
- removed joint joint_holder_1_to_plate_middle
- removed joint joint_holder_2_to_plate_middle
- removed joint joint_holder_3_to_plate_middle
- removed joint joint_holder_4_to_plate_middle
- removed joint joint_holder_5_to_plate_top
- removed joint joint_holder_6_to_plate_top
- removed joint joint_holder_7_to_plate_top
- removed joint joint_holder_8_to_plate_top
- removed joint joint_plate_bottom_to_holder_1
- removed joint joint_plate_bottom_to_holder_2
- removed joint joint_plate_bottom_to_holder_3
- removed joint joint_plate_bottom_to_holder_4
- removed joint joint_plate_middle_to_holder_5
- removed joint joint_plate_middle_to_holder_6
- removed joint joint_plate_middle_to_holder_7
- removed joint joint_plate_middle_to_holder_8
- removed joint joint_plate_top_to_screen_back
- removed joint joint_plate_top_to_screen_front
- removed joint joint_torso_to_plate_bottom
- added joint base_link_to_front_wheel: type continuous, parent base_link, child front_wheel, origin xyz=0.09 0 -0.25 rpy=0 0 0, axis 0 0 1
- added joint base_link_to_imu: type fixed, parent base_link, child imu, origin xyz=0.0 0.0 0.055 rpy=0 0 0
- added joint base_link_to_left_wheel: type continuous, parent base_link, child left_wheel, origin xyz=-0.09 -0.09 -0.25 rpy=0 0 0, axis 0 0 1
- added joint base_link_to_right_wheel: type continuous, parent base_link, child right_wheel, origin xyz=-0.09 0.09 -0.25 rpy=0 0 0, axis 0 0 1
- added joint base_to_laser: type fixed, parent base_link, child base_scan, origin xyz=0 0 0.2125 rpy=0 0 0
- added joint holder1_to_plate_middle: type fixed, parent holder1, child plate_middle, origin xyz=0 0 0.11 rpy=0 0 0
- added joint holder2_to_plate_top: type fixed, parent holder2, child plate_top, origin xyz=0 0 0.11 rpy=0 0 0
- added joint plate_bottom_to_holder1: type fixed, parent plate_bottom, child holder1, origin xyz=0 0 0.11 rpy=0 0 0
- added joint plate_middle_to_holder2: type fixed, parent plate_middle, child holder2, origin xyz=0 0 0.11 rpy=0 0 0
- added joint plate_top_to_screen_back: type fixed, parent plate_top, child screen_back, origin xyz=-0.18 0 0.02 rpy=0 0 0
- added joint plate_top_to_screen_front: type fixed, parent plate_top, child screen_front, origin xyz=0.18 0 0.02 rpy=0 0 0
- added joint screen_front_to_camera_frente: type fixed, parent screen_front, child camera_frente, origin xyz=0 0 0.11 rpy=0 0 0
- added joint torso_to_laser: type fixed, parent base_scan, child torso, origin xyz=0 0 0.2125 rpy=0 0 0
- added joint torso_to_plate: type fixed, parent torso, child plate_bottom, origin xyz=0 0 0.21 rpy=0 0 0
- joint joint_base_footprint_to_base: child base -> base_link

File: src/projeto/urdf/robot.urdf.xacro (robot description, xacro)
@@ -16,18 +16,12 @@
   <!-- Robot -->
   <xacro:base name="base_link"/>
-  <xacro:torso name="torso"/>
   <xacro:plate name="plate_bottom"/>
+  <xacro:torso name="torso" parent="base_scan" child="plate_bottom"/>
   <xacro:plate name="plate_middle"/>
   <xacro:plate name="plate_top"/>
-  <xacro:holder name="holder1" parent="plate_bottom" child="plate_middle" x= "${holder_xy}" y="${holder_xy}" z="${holder_z}"/>
-  <xacro:holder name="holder2" parent="plate_bottom" child="plate_middle" x= "${-1*holder_xy}" y="-${-1*holder_xy}" z="${holder_z}"/>
-  <xacro:holder name="holder3" parent="plate_bottom" child="plate_middle" x= "${-1*holder_xy}" y="${holder_xy}" z="${holder_z}"/>
-  <xacro:holder name="holder4" parent="plate_bottom" child="plate_middle" x= "${holder_xy}" y="${-1*holder_xy}" z="${holder_z}"/>
-  <xacro:holder name="holder5" parent="plate_middle" child="plate_top" x= "${holder_xy}" y="${holder_xy}" z="${holder_z}"/>
-  <xacro:holder name="holder6" parent="plate_middle" child="plate_top" x= "${-1*holder_xy}" y="${-1*holder_xy}" z="${holder_z}"/>
-  <xacro:holder name="holder7" parent="plate_middle" child="plate_top" x= "${-1*holder_xy}" y="${holder_xy}" z="${holder_z}"/>
-  <xacro:holder name="holder8" parent="plate_middle" child="plate_top" x= "${holder_xy}" y="${-1*holder_xy}" z="${holder_z}"/>
-  <xacro:screen name="screen_front" x="0.18" y="0" z="0.02"/>
-  <xacro:screen name="screen_back" x="-0.18" y="0" z="0.02"/>
+  <xacro:holder name="holder1" parent="plate_bottom" child="plate_middle" z="${holder_z}"/>
+  <xacro:holder name="holder2" parent="plate_middle" child="plate_top" z="${holder_z}"/>
+  <xacro:screen name="screen_front" parent="plate_top" x="0.18" y="0" z="0.02"/>
+  <xacro:screen name="screen_back" parent="plate_top" x="-0.18" y="0" z="0.02"/>
   <xacro:camera name="camera_frente" parent="screen_front" x="0" y="0" z="0.11"/>
   <xacro:wheel name="left_wheel">
@@ -36,4 +30,7 @@
   <xacro:wheel name="right_wheel">
     <origin xyz="-0.09 0.09 -0.25" rpy="0 0 0"/>
+  </xacro:wheel>
+  <xacro:wheel name="front_wheel">
+    <origin xyz="0.09 0 -0.25" rpy="0 0 0"/>
   </xacro:wheel>
   <!-- IMU -->
