Commit message: Interação verbal

File: src/projeto/urdf/macros/parts/base.urdf.xacro (robot description, xacro)
@@ -6,7 +6,7 @@
     <!-- joint: base_footprint -> base -->
     <joint name="joint_base_footprint_to_base" type="fixed">
-      <origin xyz="0 0 0.33" rpy="0 0 0"/>
+      <origin xyz="0 0 ${(wheel_radius)*2 + (laser_length)}" rpy="0 0 0"/>
       <parent link="base_footprint"/>
-      <child link="${name}"/>
+      <child link="base_scan"/>
     </joint>
     <!-- link: base -->
@@ -18,6 +18,6 @@
   <joint name="base_to_laser" type="fixed">
     <origin xyz="0 0 0.2125" rpy="0 0 0"/>
-    <parent link="${name}"/>
-    <child link="base_scan"/>
+    <parent link="base_scan"/>
+    <child link="${name}"/>
   </joint>
   <link name="base_scan">
@@ -26,4 +26,9 @@
     </xacro:create_cylinder>
   </link>
+  <joint name="base_to_plate" type="fixed">
+    <origin xyz="0 0 0.21" rpy="0 0 0"/>
+    <parent link="${name}"/>
+    <child link="plate_bottom"/>
+  </joint>
   </xacro:macro>
 </robot>

File: src/projeto/urdf/macros/parts/wheel.urdf.xacro (robot description, xacro)
@@ -5,5 +5,5 @@
     <joint name="base_link_to_${name}" type="continuous">
       <xacro:insert_block name="origin" />
-      <parent link="base_link"/>
+      <parent link="base_scan"/>
       <child link="${name}"/>
       <axis xyz="0 0 1"/>

File: src/projeto/urdf/macros/properties.urdf.xacro (robot description, xacro)
@@ -7,5 +7,5 @@
   <xacro:property name="body_length"    value="0.4" />
   <xacro:property name="laser_mass"      value="${10 * robot_mass/100}" />
-  <xacro:property name="laser_radius"    value="0.2" />
+  <xacro:property name="laser_radius"    value="${body_radius}" />
   <xacro:property name="laser_length"    value="0.025" />
   <xacro:property name="holder_mass"      value="${1.25 * robot_mass/100}" />
@@ -26,4 +26,4 @@
   <xacro:property name="camera_z"         value="0.02" />
   <xacro:property name="wheel_mass"      value="${5 * robot_mass/100}" />
-  <xacro:property name="wheel_radius"    value="${body_radius/3}" />
+  <xacro:property name="wheel_radius"    value="${body_radius/4}" />
 </robot>

File: src/projeto/urdf/robot.urdf (robot description, URDF)
Before this commit: robot garcom, 16 links, 15 joints
Links:
- removed link torso
- link front_wheel: geometry collision sphere radius=0.05; visual sphere radius=0.05
- link left_wheel: geometry collision sphere radius=0.05; visual sphere radius=0.05
- link right_wheel: geometry collision sphere radius=0.05; visual sphere radius=0.05
Joints:
- removed joint torso_to_laser
- removed joint torso_to_plate
- added joint base_to_plate: type fixed, parent base_link, child plate_bottom, origin xyz=0 0 0.21 rpy=0 0 0
- joint base_link_to_front_wheel: origin xyz=0.09 0 -0.25 rpy=0 0 0 -> xyz=0.09 0 -0.0625 rpy=0 0 0; parent base_link -> base_scan
- joint base_link_to_left_wheel: origin xyz=-0.09 -0.09 -0.25 rpy=0 0 0 -> xyz=-0.09 -0.09 -0.0625 rpy=0 0 0; parent base_link -> base_scan
- joint base_link_to_right_wheel: origin xyz=-0.09 0.09 -0.25 rpy=0 0 0 -> xyz=-0.09 0.09 -0.0625 rpy=0 0 0; parent base_link -> base_scan
- joint base_to_laser: child base_scan -> base_link; parent base_link -> base_scan
- joint joint_base_footprint_to_base: child base_link -> base_scan; origin xyz=0 0 0.33 rpy=0 0 0 -> xyz=0 0 0.125 rpy=0 0 0

File: src/projeto/urdf/robot.urdf.xacro (robot description, xacro)
@@ -8,5 +8,4 @@
   <xacro:include filename="macros/parts/plate.urdf.xacro" />
   <xacro:include filename="macros/parts/screen.urdf.xacro" />
-  <xacro:include filename="macros/parts/torso.urdf.xacro" />
   <xacro:include filename="macros/parts/wheel.urdf.xacro" />
   <xacro:include filename="simulation/gazebo_base.urdf.xacro" />
@@ -17,5 +16,4 @@
   <xacro:base name="base_link"/>
   <xacro:plate name="plate_bottom"/>
-  <xacro:torso name="torso" parent="base_scan" child="plate_bottom"/>
   <xacro:plate name="plate_middle"/>
   <xacro:plate name="plate_top"/>
@@ -26,11 +24,11 @@
   <xacro:camera name="camera_frente" parent="screen_front" x="0" y="0" z="0.11"/>
   <xacro:wheel name="left_wheel">
-    <origin xyz="-0.09 -0.09 -0.25" rpy="0 0 0"/>
+    <origin xyz="-0.09 -0.09 ${-wheel_radius -(laser_length/2)}" rpy="0 0 0"/>
   </xacro:wheel>
   <xacro:wheel name="right_wheel">
-    <origin xyz="-0.09 0.09 -0.25" rpy="0 0 0"/>
+    <origin xyz="-0.09 0.09 ${-wheel_radius -(laser_length/2)}" rpy="0 0 0"/>
   </xacro:wheel>
   <xacro:wheel name="front_wheel">
-    <origin xyz="0.09 0 -0.25" rpy="0 0 0"/>
+    <origin xyz="0.09 0 ${-wheel_radius -(laser_length/2)}" rpy="0 0 0"/>
   </xacro:wheel>
   <!-- IMU -->

File: src/projeto/urdf/simulation/gazebo_base.urdf.xacro (robot description, xacro)
@@ -15,6 +15,6 @@
         <right_joint>base_link_to_right_wheel</right_joint>
         <!-- kinematics -->
-        <wheel_separation>0.025</wheel_separation>
-        <wheel_diameter>0.13</wheel_diameter>
+        <wheel_separation>0.13</wheel_separation>
+        <wheel_diameter>0.1</wheel_diameter>
         <!-- limits -->
         <max_wheel_torque>20</max_wheel_torque>
