Commit message: urdf tcc

File: src/tcc/urdf/macros/parts/base.urdf.xacro (robot description, xacro)
@@ -6,7 +6,7 @@
     <!-- joint: base_footprint -> base -->
     <joint name="joint_base_footprint_to_base" type="fixed">
-      <origin xyz="0 0 ${(wheel_radius)*2 + (laser_length)}" rpy="0 0 0"/>
+      <origin xyz="0 0 ${(wheel_radius)*2}" rpy="0 0 0"/>
       <parent link="base_footprint"/>
-      <child link="base_scan"/>
+      <child link="base_link"/>
     </joint>
     <!-- link: base -->
@@ -17,5 +17,5 @@
     </link>
   <joint name="base_to_laser" type="fixed">
-    <origin xyz="0 0 0.2125" rpy="0 0 0"/>
+    <origin xyz="0 0 ${body_length/2 + laser_length/2}" rpy="0 0 0"/>
     <parent link="base_scan"/>
     <child link="${name}"/>
@@ -26,9 +26,4 @@
     </xacro:create_cylinder>
   </link>
-  <joint name="base_to_plate" type="fixed">
-    <origin xyz="0 0 0.21" rpy="0 0 0"/>
-    <parent link="${name}"/>
-    <child link="plate_bottom"/>
-  </joint>
   </xacro:macro>
 </robot>

File: src/tcc/urdf/macros/properties.urdf.xacro (robot description, xacro)
@@ -2,28 +2,12 @@
 <robot xmlns:xacro="http://ros.org/wiki/xacro">
   <xacro:property name="PI"             value="3.14159265" />
-  <xacro:property name="robot_mass"      value="10" />
-  <xacro:property name="body_mass"      value="${20 * robot_mass/100}" />
-  <xacro:property name="body_radius"    value="0.2" />
-  <xacro:property name="body_length"    value="0.4" />
-  <xacro:property name="laser_mass"      value="${10 * robot_mass/100}" />
-  <xacro:property name="laser_radius"    value="${body_radius}" />
+  <xacro:property name="robot_mass"      value="3" />
+  <xacro:property name="body_mass"      value="${70 * robot_mass/100}" />
+  <xacro:property name="body_radius"    value="0.115" />
+  <xacro:property name="body_length"    value="0.2" />
+  <xacro:property name="laser_mass"      value="${15 * robot_mass/100}" />
+  <xacro:property name="laser_radius"    value="${body_radius/3}" />
   <xacro:property name="laser_length"    value="0.025" />
-  <xacro:property name="holder_mass"      value="${1.25 * robot_mass/100}" />
-  <xacro:property name="holder_radius"    value="0.02" />
-  <xacro:property name="holder_length"    value="0.2" />
-  <xacro:property name="holder_xy"        value="0.12" />
-  <xacro:property name="holder_z"         value="0.11" />
-  <xacro:property name="plate_mass"      value="${5 * robot_mass/100}" />
-  <xacro:property name="plate_radius"    value="${body_radius}" />
-  <xacro:property name="plate_length"    value="0.02" />
-  <xacro:property name="screen_mass"      value="${4 * robot_mass/100}" />
-  <xacro:property name="screen_x"         value="0.05" />
-  <xacro:property name="screen_y"         value="0.2" />
-  <xacro:property name="screen_z"         value="0.2" />
-  <xacro:property name="camera_mass"      value="${2 * robot_mass/100}" />
-  <xacro:property name="camera_x"         value="0.025" />
-  <xacro:property name="camera_y"         value="0.025" />
-  <xacro:property name="camera_z"         value="0.02" />
   <xacro:property name="wheel_mass"      value="${5 * robot_mass/100}" />
-  <xacro:property name="wheel_radius"    value="${body_radius/4}" />
+  <xacro:property name="wheel_radius"    value="0.0335" />
 </robot>

File: src/tcc/urdf/robot.urdf.xacro (robot description, xacro)
@@ -1,11 +1,7 @@
 <?xml version="1.0"?>
-<robot name="garcom" xmlns:xacro="http://www.ros.org/wiki/xacro">
+<robot name="limpeza" xmlns:xacro="http://www.ros.org/wiki/xacro">
   <xacro:include filename="macros/link_geometry.urdf.xacro" />
   <xacro:include filename="macros/properties.urdf.xacro" />
   <xacro:include filename="macros/parts/base.urdf.xacro" />
-  <xacro:include filename="macros/parts/camera.urdf.xacro" />
-  <xacro:include filename="macros/parts/holder.urdf.xacro" />
-  <xacro:include filename="macros/parts/plate.urdf.xacro" />
-  <xacro:include filename="macros/parts/screen.urdf.xacro" />
   <xacro:include filename="macros/parts/wheel.urdf.xacro" />
   <xacro:include filename="simulation/gazebo_base.urdf.xacro" />
@@ -15,28 +11,19 @@
   <!-- Robot -->
   <xacro:base name="base_link"/>
-  <xacro:plate name="plate_bottom"/>
-  <xacro:plate name="plate_middle"/>
-  <xacro:plate name="plate_top"/>
-  <xacro:holder name="holder1" parent="plate_bottom" child="plate_middle" z="${holder_z}"/>
-  <xacro:holder name="holder2" parent="plate_middle" child="plate_top" z="${holder_z}"/>
-  <xacro:screen name="screen_front" parent="plate_top" x="0.18" y="0" z="0.02"/>
-  <xacro:screen name="screen_back" parent="plate_top" x="-0.18" y="0" z="0.02"/>
-  <xacro:camera name="camera_frente" parent="screen_front" x="0" y="0" z="0.11"/>
   <xacro:wheel name="left_wheel">
-    <origin xyz="-0.09 -0.09 ${-wheel_radius -(laser_length/2)}" rpy="0 0 0"/>
+    <origin xyz="-0.048 -0.048 ${-wheel_radius}" rpy="0 0 0"/>
   </xacro:wheel>
   <xacro:wheel name="right_wheel">
-    <origin xyz="-0.09 0.09 ${-wheel_radius -(laser_length/2)}" rpy="0 0 0"/>
+    <origin xyz="-0.048 0.048 ${-wheel_radius}" rpy="0 0 0"/>
   </xacro:wheel>
   <xacro:wheel name="front_wheel">
-    <origin xyz="0.09 0 ${-wheel_radius -(laser_length/2)}" rpy="0 0 0"/>
+    <origin xyz="0.048 0 ${-wheel_radius}" rpy="0 0 0"/>
   </xacro:wheel>
-  <!-- IMU -->
+  <!-- IMU
   <xacro:imu name="imu" parent="base_link">
     <origin xyz="0.0 0.0 0.055" rpy="0 0 0"/>
-  </xacro:imu>
+  </xacro:imu> -->
   <!-- Plugins -->
   <xacro:gazebo_base/>
   <xacro:gazebo_laser reference="base_scan"/>
-  <xacro:gazebo_camera reference="camera_frente"/>
 </robot>

File: src/tcc/urdf/simulation/gazebo_base.urdf.xacro (robot description, xacro)
@@ -15,6 +15,6 @@
         <right_joint>base_link_to_right_wheel</right_joint>
         <!-- kinematics -->
-        <wheel_separation>0.13</wheel_separation>
-        <wheel_diameter>0.1</wheel_diameter>
+        <wheel_separation>0.09</wheel_separation>
+        <wheel_diameter>0.067</wheel_diameter>
         <!-- limits -->
         <max_wheel_torque>20</max_wheel_torque>
