Commit message: fix simulation

File: src/tcc/urdf/macros/parts/wheel.urdf.xacro (robot description, xacro)
@@ -7,5 +7,5 @@
       <parent link="base_scan"/>
       <child link="${name}"/>
-      <axis xyz="0 1 0"/>
+      <axis xyz="0 0 1"/>
     </joint>
     <!-- link: wheel -->

File: src/tcc/urdf/robot.urdf.xacro (robot description, xacro)
@@ -24,8 +24,8 @@
   <xacro:camera name="camera_frente" parent="screen_front" x="0" y="0" z="0.11"/>
   <xacro:wheel name="left_wheel">
-    <origin xyz="-0.09 0.09 ${-wheel_radius -(laser_length/2)}" rpy="0 0 0"/>
+    <origin xyz="-0.09 -0.09 ${-wheel_radius -(laser_length/2)}" rpy="0 0 0"/>
   </xacro:wheel>
   <xacro:wheel name="right_wheel">
-    <origin xyz="-0.09 -0.09 ${-wheel_radius -(laser_length/2)}" rpy="0 0 0"/>
+    <origin xyz="-0.09 0.09 ${-wheel_radius -(laser_length/2)}" rpy="0 0 0"/>
   </xacro:wheel>
   <xacro:wheel name="front_wheel">

Commit message: Fixed Tcc urdf

File: src/tcc/urdf/macros/parts/wheel.urdf.xacro (robot description, xacro)
@@ -7,5 +7,5 @@
       <parent link="base_link"/>
       <child link="${name}"/>
-      <axis xyz="0 0 1"/>
+      <axis xyz="0 1 0"/>
     </joint>
     <!-- link: wheel -->

File: src/tcc/urdf/robot.urdf (robot description, URDF)
Before this commit: robot limpeza, 6 links, 5 joints
Joints:
- joint base_link_to_front_wheel: origin xyz=0.048 0 -0.0335 rpy=0 0 0 -> xyz=0.048 0 -0.1335 rpy=0 0 0

File: src/tcc/urdf/robot.urdf.xacro (robot description, xacro)
@@ -12,8 +12,8 @@
   <xacro:base name="base_link"/>
   <xacro:wheel name="left_wheel">
-    <origin xyz="-0.048 -0.048 ${-wheel_radius -body_length/2}" rpy="0 0 0"/>
+    <origin xyz="-0.048 0.048 ${-wheel_radius -body_length/2}" rpy="0 0 0"/>
   </xacro:wheel>
   <xacro:wheel name="right_wheel">
-    <origin xyz="-0.048 0.048 ${-wheel_radius -body_length/2}" rpy="0 0 0"/>
+    <origin xyz="-0.048 -0.048 ${-wheel_radius -body_length/2}" rpy="0 0 0"/>
   </xacro:wheel>
   <xacro:wheel name="front_wheel">

File: src/tcc/urdf/simulation/gazebo_base.urdf.xacro (robot description, xacro)
@@ -15,5 +15,5 @@
         <right_joint>base_link_to_right_wheel</right_joint>
         <!-- kinematics -->
-        <wheel_separation>0.09</wheel_separation>
+        <wheel_separation>0.096</wheel_separation>
         <wheel_diameter>0.067</wheel_diameter>
         <!-- limits -->

File: src/tcc/urdf/simulation/gazebo_laser.urdf.xacro (robot description, xacro)
@@ -14,5 +14,5 @@
         </scan>
         <range>
-          <min>0.5</min>
+          <min>0.2</min>
           <max>30.0</max>
           <resolution>0.015000</resolution>
