Commit message: urdf tcc

File: src/projeto/urdf/macros/properties.urdf.xacro (robot description, xacro)
@@ -3,23 +3,23 @@
   <xacro:property name="PI"             value="3.14159265" />
   <xacro:property name="robot_mass"      value="10" />
-  <xacro:property name="body_mass"      value="${20 * robot_mass/100}" />
-  <xacro:property name="body_radius"    value="0.2" />
+  <xacro:property name="body_mass"      value="${10 * robot_mass/100}" />
+  <xacro:property name="body_radius"    value="0.3" />
   <xacro:property name="body_length"    value="0.4" />
-  <xacro:property name="laser_mass"      value="${10 * robot_mass/100}" />
+  <xacro:property name="laser_mass"      value="${50 * robot_mass/100}" />
   <xacro:property name="laser_radius"    value="${body_radius}" />
   <xacro:property name="laser_length"    value="0.025" />
-  <xacro:property name="holder_mass"      value="${1.25 * robot_mass/100}" />
+  <xacro:property name="holder_mass"      value="${5 * robot_mass/100}" />
   <xacro:property name="holder_radius"    value="0.02" />
   <xacro:property name="holder_length"    value="0.2" />
   <xacro:property name="holder_xy"        value="0.12" />
   <xacro:property name="holder_z"         value="0.11" />
-  <xacro:property name="plate_mass"      value="${5 * robot_mass/100}" />
+  <xacro:property name="plate_mass"      value="${4 * robot_mass/100}" />
   <xacro:property name="plate_radius"    value="${body_radius}" />
   <xacro:property name="plate_length"    value="0.02" />
-  <xacro:property name="screen_mass"      value="${4 * robot_mass/100}" />
+  <xacro:property name="screen_mass"      value="${1 * robot_mass/100}" />
   <xacro:property name="screen_x"         value="0.05" />
   <xacro:property name="screen_y"         value="0.2" />
   <xacro:property name="screen_z"         value="0.2" />
-  <xacro:property name="camera_mass"      value="${2 * robot_mass/100}" />
+  <xacro:property name="camera_mass"      value="${1 * robot_mass/100}" />
   <xacro:property name="camera_x"         value="0.025" />
   <xacro:property name="camera_y"         value="0.025" />

File: src/projeto/urdf/robot.urdf (robot description, URDF)
Before this commit: robot garcom, 15 links, 14 joints
Links:
- added link front_wheel2, mass 0.5; collision sphere radius=0.075; visual sphere radius=0.075
- link base_link: mass 2.0 -> 1.0; geometry collision cylinder length=0.4 radius=0.3; visual cylinder length=0.4 radius=0.3
- link base_scan: mass 1.0 -> 5.0; geometry collision cylinder length=0.025 radius=0.3; visual cylinder length=0.025 radius=0.3
- link camera_frente: mass 0.2 -> 0.1
- link front_wheel: geometry collision sphere radius=0.075; visual sphere radius=0.075
- link holder1: mass 0.125 -> 0.5
- link holder2: mass 0.125 -> 0.5
- link left_wheel: geometry collision sphere radius=0.075; visual sphere radius=0.075
- link plate_bottom: mass 0.5 -> 0.4; geometry collision cylinder length=0.02 radius=0.3; visual cylinder length=0.02 radius=0.3
- link plate_middle: mass 0.5 -> 0.4; geometry collision cylinder length=0.02 radius=0.3; visual cylinder length=0.02 radius=0.3
- link plate_top: mass 0.5 -> 0.4; geometry collision cylinder length=0.02 radius=0.3; visual cylinder length=0.02 radius=0.3
- link right_wheel: geometry collision sphere radius=0.075; visual sphere radius=0.075
- link screen_back: mass 0.4 -> 0.1
- link screen_front: mass 0.4 -> 0.1
Joints:
- added joint base_link_to_front_wheel2: type continuous, parent base_scan, child front_wheel2, origin xyz=0.16 -0.16 -0.0875 rpy=0 0 0, axis 0 1 0
- joint base_link_to_front_wheel: axis 0 0 1 -> 0 1 0; origin xyz=0.09 0 -0.0625 rpy=0 0 0 -> xyz=0.16 0.16 -0.0875 rpy=0 0 0
- joint base_link_to_left_wheel: axis 0 0 1 -> 0 1 0; origin xyz=-0.09 -0.09 -0.0625 rpy=0 0 0 -> xyz=-0.16 0.16 -0.0875 rpy=0 0 0
- joint base_link_to_right_wheel: axis 0 0 1 -> 0 1 0; origin xyz=-0.09 0.09 -0.0625 rpy=0 0 0 -> xyz=-0.16 -0.16 -0.0875 rpy=0 0 0
- joint joint_base_footprint_to_base: origin xyz=0 0 0.125 rpy=0 0 0 -> xyz=0 0 0.175 rpy=0 0 0
- joint plate_top_to_screen_back: origin xyz=-0.18 0 0.02 rpy=0 0 0 -> xyz=-0.3 0 0.02 rpy=0 0 0
- joint plate_top_to_screen_front: origin xyz=0.18 0 0.02 rpy=0 0 0 -> xyz=0.3 0 0.02 rpy=0 0 0

File: src/projeto/urdf/robot.urdf.xacro (robot description, xacro)
@@ -20,15 +20,18 @@
   <xacro:holder name="holder1" parent="plate_bottom" child="plate_middle" z="${holder_z}"/>
   <xacro:holder name="holder2" parent="plate_middle" child="plate_top" z="${holder_z}"/>
-  <xacro:screen name="screen_front" parent="plate_top" x="0.18" y="0" z="0.02"/>
-  <xacro:screen name="screen_back" parent="plate_top" x="-0.18" y="0" z="0.02"/>
+  <xacro:screen name="screen_front" parent="plate_top" x="0.3" y="0" z="0.02"/>
+  <xacro:screen name="screen_back" parent="plate_top" x="-0.3" y="0" z="0.02"/>
   <xacro:camera name="camera_frente" parent="screen_front" x="0" y="0" z="0.11"/>
   <xacro:wheel name="left_wheel">
-    <origin xyz="-0.09 0.09 ${-wheel_radius -(laser_length/2)}" rpy="0 0 0"/>
+    <origin xyz="-0.16 0.16 ${-wheel_radius -(laser_length/2)}" rpy="0 0 0"/>
   </xacro:wheel>
   <xacro:wheel name="right_wheel">
-    <origin xyz="-0.09 -0.09 ${-wheel_radius -(laser_length/2)}" rpy="0 0 0"/>
+    <origin xyz="-0.16 -0.16 ${-wheel_radius -(laser_length/2)}" rpy="0 0 0"/>
   </xacro:wheel>
   <xacro:wheel name="front_wheel">
-    <origin xyz="0.09 0 ${-wheel_radius -(laser_length/2)}" rpy="0 0 0"/>
+    <origin xyz="0.16 0.16 ${-wheel_radius -(laser_length/2)}" rpy="0 0 0"/>
+  </xacro:wheel>
+  <xacro:wheel name="front_wheel2">
+    <origin xyz="0.16 -0.16 ${-wheel_radius -(laser_length/2)}" rpy="0 0 0"/>
   </xacro:wheel>
   <!-- IMU -->

File: src/projeto/urdf/simulation/gazebo_base.urdf.xacro (robot description, xacro)
@@ -15,6 +15,6 @@
         <right_joint>base_link_to_right_wheel</right_joint>
         <!-- kinematics -->
-        <wheel_separation>0.13</wheel_separation>
-        <wheel_diameter>0.1</wheel_diameter>
+        <wheel_separation>0.32</wheel_separation>
+        <wheel_diameter>0.15</wheel_diameter>
         <!-- limits -->
         <max_wheel_torque>20</max_wheel_torque>

File: src/tcc/urdf/macros/parts/base.urdf.xacro (robot description, xacro)
@@ -18,6 +18,6 @@
   <joint name="base_to_laser" type="fixed">
     <origin xyz="0 0 ${body_length/2 + laser_length/2}" rpy="0 0 0"/>
-    <parent link="base_scan"/>
-    <child link="${name}"/>
+    <parent link="${name}"/>
+    <child link="base_scan"/>
   </joint>
   <link name="base_scan">

File: src/tcc/urdf/macros/parts/wheel.urdf.xacro (robot description, xacro)
@@ -5,5 +5,5 @@
     <joint name="base_link_to_${name}" type="continuous">
       <xacro:insert_block name="origin" />
-      <parent link="base_scan"/>
+      <parent link="base_link"/>
       <child link="${name}"/>
       <axis xyz="0 0 1"/>

File: src/tcc/urdf/robot.urdf (robot description, URDF)
Before this commit: robot garcom, 15 links, 14 joints
Links:
- removed link camera_frente
- removed link holder1
- removed link holder2
- removed link imu
- removed link plate_bottom
- removed link plate_middle
- removed link plate_top
- removed link screen_back
- removed link screen_front
- link base_link: mass 2.0 -> 2.1; geometry collision cylinder length=0.2 radius=0.115; visual cylinder length=0.2 radius=0.115
- link base_scan: mass 1.0 -> 0.45; geometry collision cylinder length=0.025 radius=0.03833333333333334; visual cylinder length=0.025 radius=0.03833333333333334
- link front_wheel: mass 0.5 -> 0.15; geometry collision sphere radius=0.0335; visual sphere radius=0.0335
- link left_wheel: mass 0.5 -> 0.15; geometry collision sphere radius=0.0335; visual sphere radius=0.0335
- link right_wheel: mass 0.5 -> 0.15; geometry collision sphere radius=0.0335; visual sphere radius=0.0335
Joints:
- removed joint base_link_to_imu
- removed joint base_to_plate
- removed joint holder1_to_plate_middle
- removed joint holder2_to_plate_top
- removed joint plate_bottom_to_holder1
- removed joint plate_middle_to_holder2
- removed joint plate_top_to_screen_back
- removed joint plate_top_to_screen_front
- removed joint screen_front_to_camera_frente
- joint base_link_to_front_wheel: origin xyz=0.09 0 -0.0625 rpy=0 0 0 -> xyz=0.048 0 -0.0335 rpy=0 0 0; parent base_scan -> base_link
- joint base_link_to_left_wheel: origin xyz=-0.09 -0.09 -0.0625 rpy=0 0 0 -> xyz=-0.048 -0.048 -0.1335 rpy=0 0 0; parent base_scan -> base_link
- joint base_link_to_right_wheel: origin xyz=-0.09 0.09 -0.0625 rpy=0 0 0 -> xyz=-0.048 0.048 -0.1335 rpy=0 0 0; parent base_scan -> base_link
- joint base_to_laser: child base_link -> base_scan; origin xyz=0 0 0.2125 rpy=0 0 0 -> xyz=0 0 0.1125 rpy=0 0 0; parent base_scan -> base_link
- joint joint_base_footprint_to_base: child base_scan -> base_link; origin xyz=0 0 0.125 rpy=0 0 0 -> xyz=0 0 0.067 rpy=0 0 0

File: src/tcc/urdf/robot.urdf.xacro (robot description, xacro)
@@ -12,11 +12,11 @@
   <xacro:base name="base_link"/>
   <xacro:wheel name="left_wheel">
-    <origin xyz="-0.048 -0.048 ${-wheel_radius}" rpy="0 0 0"/>
+    <origin xyz="-0.048 -0.048 ${-wheel_radius -body_length/2}" rpy="0 0 0"/>
   </xacro:wheel>
   <xacro:wheel name="right_wheel">
-    <origin xyz="-0.048 0.048 ${-wheel_radius}" rpy="0 0 0"/>
+    <origin xyz="-0.048 0.048 ${-wheel_radius -body_length/2}" rpy="0 0 0"/>
   </xacro:wheel>
   <xacro:wheel name="front_wheel">
-    <origin xyz="0.048 0 ${-wheel_radius}" rpy="0 0 0"/>
+    <origin xyz="0.048 0 ${-wheel_radius -body_length/2}" rpy="0 0 0"/>
   </xacro:wheel>
   <!-- IMU
