Commit message: working on simulation

File: src/projeto/urdf/robot.urdf (robot description, URDF)
Before this commit: robot garcom, 20 links, 25 joints
Links:
- link torso: geometry collision cylinder length=0.3 radius=0.2; visual cylinder length=0.4 radius=0.2

Commit message: fixed tcc simulation, missing checkpoints nav

File: src/projeto/urdf/robot.urdf (robot description, URDF)
Before this commit: robot garcom, 16 links, 15 joints
Links:
- removed link camera_frente
- removed link imu
Joints:
- removed joint base_link_to_imu
- removed joint screen_front_to_camera_frente

File: src/tcc/urdf/robot.urdf.xacro (robot description, xacro)
@@ -20,8 +20,8 @@
     <origin xyz="0.048 0 ${-wheel_radius -body_length/2}" rpy="0 0 0"/>
   </xacro:wheel>
-  <!-- IMU
+  <!-- IMU -->
   <xacro:imu name="imu" parent="base_link">
     <origin xyz="0.0 0.0 0.055" rpy="0 0 0"/>
-  </xacro:imu> -->
+  </xacro:imu>
   <!-- Plugins -->
   <xacro:gazebo_base/>

File: src/tcc/urdf/simulation/gazebo_laser.urdf.xacro (robot description, xacro)
@@ -9,10 +9,10 @@
             <samples>180</samples>
             <resolution>1.0</resolution>
-            <min_angle>-1.57</min_angle>
-            <max_angle>1.57</max_angle>
+            <min_angle>-3.14</min_angle>
+            <max_angle>3.14</max_angle>
           </horizontal>
         </scan>
         <range>
-          <min>0.2</min>
+          <min>0.1</min>
           <max>30.0</max>
           <resolution>0.015000</resolution>

File: src/tcc/urdf/simulation/imu.urdf.xacro (robot description, xacro)
@@ -10,10 +10,10 @@
       <visual>
         <geometry>
-          <box size="0.2 0.2 0.05"/>
+          <box size="0.02 0.02 0.05"/>
         </geometry>
       </visual>
       <collision>
         <geometry>
-          <box size="0.2 0.2 0.05"/>
+          <box size="0.02 0.02 0.05"/>
         </geometry>
       </collision>
